File: Design/H00R3.sch (EAGLE design)
At the start: 2 parts, among them P1 HEXABIT_17.32

Commit message: -Fix some schematic issues
Other:
- note added: "H00R3_Frontend"
- note removed: "H00R3_Backend"
Changed lines of the file:
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@@
 <text x="180.9242" y="19.6342" size="1.9304" layer="102" font="vector">H00R3</text>
 <text x="191.9478" y="11.2014" size="1.9304" layer="101" font="vector" align="center">Horizontal Extension (Spacer)</text>
-<text x="206.3242" y="19.6342" size="1.9304" layer="101" font="vector">H00R3_Backend</text>
+<text x="206.3242" y="19.6342" size="1.9304" layer="101" font="vector">H00R3_Frontend</text>
 <wire x1="168.91" y1="3.81" x2="168.91" y2="8.128" width="0.1524" layer="205"/>
 <wire x1="168.91" y1="8.128" x2="168.91" y2="18.288" width="0.1524" layer="205"/>
